File: eagle/ElectromagPWM/electromag_pwm.brd (EAGLE design)
At the start: 36.5 x 68.6 mm, 14 parts, among them IC1 NE555, Q1 SUP75N06

Commit message: board changes and neopixel
Parts:
- moved D1 16.7 mm to (35.6, 63.5)
- moved R3 15.9 mm to (22.9, 63.5)
- moved D2 6.84 mm to (31.8, 53.3)
- moved Q1 6.84 mm to (33.0, 16.5)
- moved R1 6.84 mm to (15.2, 53.3)
- moved C2 6.84 mm to (30.5, 43.2)
- moved D3 6.84 mm to (17.8, 19.1)
- moved D4 6.84 mm to (17.8, 25.4)
- moved D5 6.84 mm to (17.8, 31.8)
- moved IC1 6.84 mm to (19.1, 41.9)
- moved JP2 6.84 mm to (17.8, 11.4)
- moved JP1 6.84 mm to (15.2, 63.5)
- moved C1 6.84 mm to (22.9, 50.8)
- moved R2 6.84 mm to (25.4, 58.4)
Routing:
- net VCC: track 31.9 -> 97.3 mm
- net GND: track 107.7 -> 155.5 mm
- net N$7: track 32.6 -> 52.3 mm
- net N$6: track 92.8 -> 78.0 mm
- net N$3: track 5.65 -> 13.5 mm
- net PWM: track 54.1 -> 53.3 mm
- net INDUCTOR_NEG: track 37.0 -> 37.7 mm
- added copper zone on layer 16, net GND
Other:
- board size 36.5 x 68.6 mm -> 100 x 80 mm
- board text added: "ElectroGlad"
